Commit message: Learning code for 3 blocks

File: bullet3/examples/pybullet/gym/pybullet_data/block.urdf (robot description, URDF)
Before this commit: robot block_2, 1 links, 0 joints
Links:
- link block_2_base_link: geometry collision box size=0 0 0; visual box size=0.10 0.018 0.018

File: bullet3/examples/pybullet/gym/pybullet_data/block1.urdf (robot description, URDF)
Before this commit: robot block_2, 1 links, 0 joints
Links:
- link block_2_base_link: geometry collision box size=0 0 0; visual box size=0.10 0.018 0.018

File: bullet3/examples/pybullet/gym/pybullet_data/block2.urdf (robot description, URDF)
Before this commit: robot block_2, 1 links, 0 joints
Links:
- link block_2_base_link: geometry collision box size=0 0 0; visual box size=0.10 0.018 0.018

Commit message: Testing kuka

File: bullet3/examples/pybullet/gym/pybullet_data/block.urdf (robot description, URDF)
Before this commit: robot block_2, 1 links, 0 joints
Links:
- link block_2_base_link: geometry collision box size=0 0 0; visual box size=0.1 0.1 0.1

File: bullet3/examples/pybullet/gym/pybullet_data/block1.urdf (robot description, URDF)
Before this commit: robot block_2, 1 links, 0 joints
Links:
- link block_2_base_link: geometry collision box size=0 0 0; visual box size=0.1 0.1 0.1

File: bullet3/examples/pybullet/gym/pybullet_data/block2.urdf (robot description, URDF)
Before this commit: robot block_2, 1 links, 0 joints
Links:
- link block_2_base_link: geometry collision box size=0 0 0; visual box size=0.1 0.1 0.1
